File: KiCad/SpUnLy58.kicad_pcb (KiCad board)
At the start: 2 copper layers, 318.8 x 137.2 mm, 131 parts

Commit message: tuned tracks, moved mounting hole.
Parts:
- moved _10 1.32 mm to (225.4, 133.2)
- moved _9 0.91 mm to (164.4, 133.2)
- moved D19 0.34 mm to (141.7, 119.1)
- moved S27 0.34 mm to (118.2, 165.5)
- moved D44 0.34 mm to (279.3, 97.9)
- moved D26 0.34 mm to (105.2, 164.3)
- moved S3 0.34 mm to (51.1, 99.9)
- moved S34 0.34 mm to (323.3, 135.7)
- moved S49 0.34 mm to (247.5, 95.6)
- moved _5 0.34 mm to (82.4, 147.0)
- moved S30 0.34 mm to (342.4, 135.7)
- moved S56 0.34 mm to (271.5, 165.5)
- moved D50 0.34 mm to (260.0, 155.0)
- moved S12 0.34 mm to (104.0, 79.2)
- moved D37 0.34 mm to (324.5, 85.1)
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Routing:
- net P106: track 212.8 -> 205.7 mm
- net P008: track 522.8 -> 522.2 mm

Commit message: Version 1.0 complete. Finalized routes. Added graphics.
Parts:
- added G***: LOGO, temp:giraffasax-logo, F.Cu at (223.6, 83.8)
Other:
- board text added: "SpUnLy58 v1.0 by Giraffasax"

Commit message: [v1.1] Reduced vertical spacing from 18 to 17mm Fixed jstph connector footprint and pad label. Increased cutout for battery.
Parts:
- moved JST1 15.2 mm to (221.3, 136.9), turned to -90 degrees
- moved S53 10.3 mm to (239.1, 106.4)
- moved D53 10.3 mm to (248.3, 106.7)
- moved D49 10.2 mm to (266.8, 97.3)
- moved S49 10.2 mm to (257.6, 96.7)
- moved S45 10.1 mm to (274.0, 81.1)
- moved D45 10.1 mm to (283.2, 82.1)
- moved S41 10.0 mm to (295.7, 80.4)
- moved D41 10.0 mm to (304.7, 81.6)
- moved D5 9.98 mm to (83.9, 139.1)
- moved S13 9.98 mm to (117.1, 129.1)
- moved D1 9.98 mm to (64.9, 138.9)
- moved _5 9.98 mm to (92.2, 145.3)
- moved D26 9.98 mm to (115.1, 162.7)
- moved S5 9.98 mm to (76.3, 134.0)
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Connections:
- JST1 pad 1: pos -> GND
- JST1 pad 2: GND -> pos
Routing:
- net P002: track 405.2 -> 381.0 mm
- net P101: track 164.8 -> 182.4 mm
- net P029: track 467.1 -> 457.1 mm
- net P008: track 522.2 -> 530.2 mm
- net P009: track 195.9 -> 188.4 mm
- net pos: track 66.4 -> 73.2 mm
- net P031: track 504.9 -> 498.3 mm
- net GND: track 103.2 -> 107.9 mm
- net VCC: track 49.3 -> 45.1 mm
- net P022: track 597.3 -> 601.2 mm
- net P113: track 199.6 -> 202.2 mm
- net P024: track 546.5 -> 544.3 mm
- net RST: track 31.3 -> 33.4 mm
- net P111: track 210.1 -> 212.1 mm
- net P104: track 195.2 -> 193.2 mm
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Other:
- board size 318.8 x 137.2 mm -> 318 x 134.4 mm
- board text added: "Off <-> On"
- board text added: "SpUnLy58 v1.1 by Giraffasax"
- board text removed: "SpUnLy58 v1.0 by Giraffasax"
